File: envirodinges.sch (EAGLE design)
At the start: 32 parts, among them IC1 W5500_MODULE, T1 IRF520(V), U1 MODULE_TCA9548, U2 R-78B5.0-1.0(V), U3 R-78B3.3-1.0(V), X1 MKDSN1,5/4-5,08, X5 MKDSN1,5/3-5,08

Commit message: Add files via upload
Parts:
- added LED5, LED6: (no value), led-rs:LED-3MM
- added R8, R9: (no value), rcl-rs:R-EU0207/10
Connections:
- net N$20 renamed ACTIVE_LED
- net N$22 renamed ERROR_LED
- new net N$2: LED6.A, R9.1
- new net SS: B1.7, IC1./SS
- net +5V: now also R9.2
- net GND: now also B1.4, LED6.C
Other:
- note added: "D4 low - Container 1 D4 high - Container 2 D4 set as input-pullup"
- moved on the sheet: C2, C5, D1, R5, R6, R7, U3, X5-1, X5-2, X5-3, X6

Commit message: Add files via upload
TTL<->RS232 module met echte DB9 connector
Parts:
- removed G1: MODULE_MAX3232, diy-modules:MODULE_MAX3232
- removed X5: MKDSN1,5/3-5,08, con-phoenix-508:MKDSN1,5/3-5,08
- added U4: MODULE_MAX3232_DB9, diy-modules:MODULE_MAX3232_DB9
- C1: value (none) -> 47u/40V
- C2, C3, C4, C5: value (none) -> 10u/16V
- LED1, LED4, LED5: value (none) -> gn
- LED2: value (none) -> bl
- LED3: value (none) -> red
- R1, R2: value (none) -> 2k2
- R3, R4, R7: value (none) -> 10k
- R5, R6, R9: value (none) -> 270
- R8: value (none) -> 180
- RN1: value (none) -> 4k7
Connections:
- removed net RS232_RX: G1.RX_R, X5-3.KL
- removed net RS232_TX: G1.TX_R, X5-1.KL
- new net N$4: LED5.C, R8.2
- net +3V3: now also LED5.A
- net +5V: now also U4.VCC; no longer G1.VCC
- net GND: now also R8.1, U4.GND; no longer G1.GND, X5-2.KL
- net N$15: now also U4.TX_T; no longer G1.TX_T
- net N$16: now also U4.RX_T; no longer G1.RX_T
Other:
- moved on the sheet: C4, IC1, LED5, R3, R4, R7, R8

Commit message: Ander RS232 module
Parts:
- removed X6: (no value), con-phoenix-254:MPT3
- added X5, X7: MKDSN1,5/3-5,08, con-phoenix-508:MKDSN1,5/3-5,08
- LED3: value red -> rd
- R5, R6: value 270 -> 220
- U4: value MODULE_MAX3232_DB9 -> MODULE_MAX3232-B; device diy-modules:MODULE_MAX3232_DB9 -> diy-modules:MODULE_MAX3232-B
Connections:
- new net N$3: U4.RX_R, X5-3.KL
- new net N$5: U4.TX_R, X5-2.KL
- net ACTIVE_LED: now also X7-1.KL; no longer X6.1
- net ERROR_LED: now also X7-3.KL; no longer X6.3
- net GND: now also X5-1.KL, X7-2.KL; no longer X6.2
Other:
- moved on the sheet: C3, LED3, LED4, RN1, U1, X2, X3, X4
